File: Hardware/MCU/MCU.kicad_sch (KiCad schematic)
At the start: 35 parts, among them J1 spi0, J10 i2s, J11 USB_C_Receptacle_USB2.0_16P, J2 sp1, J3 sp2, J4 1778612, J5 1778612, J6 1778612, J7 1778612, J8 i2c0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

Commit message: text aangepast
Other:
- note added: "1.0"
- note added: "3-4-2025"
- note added: "MCU PCB"
Changed lines of the file:
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@@
+		)
+	)
+	(text "1.0\n\n"
+		(exclude_from_sim no)
+		(at 270.764 194.564 0)
+		(effects
+			(font
+				(size 1.27 1.27)
+			)
+		)
+	)
+	(text "MCU PCB\n"
+		(exclude_from_sim no)
+		(at 192.278 189.738 0)
+		(effects
+			(font
+				(size 1.27 1.27)
+			)
 		)
 	)
@@
 		(effects
 			(font
+				(size 1.27 1.27)
+			)
+		)
+	)
+	(text "3-4-2025\n"
+		(exclude_from_sim no)
+		(at 212.09 193.548 0)
+		(effects
+			(font
